Commit message: modify urdf for mini with rplidar a2 and realsense d435i

File: handsfree_gazebo/urdf_stone_v3/common_properties.xacro (robot description, xacro)
@@ -1,4 +1,5 @@
 <?xml version="1.0"?>
 <robot name="xacro_properties" xmlns:xacro="http://www.ros.org/wiki/xacro">
+  <xacro:property name="M_PI" value="3.1415926535897931" />
   <!-- Init colour -->
   <material name="black">

File: handsfree_gazebo/urdf_stone_v3/stone_v3_base.xacro (robot description, xacro)
@@ -7,293 +7,325 @@
   <xacro:include filename="$(find handsfree_gazebo)/urdf_stone_v3/common_properties.xacro"/>
   <xacro:macro name="stone_v3_base">
-  <link name="base_footprint"/>
-  <link name="base_link">
-    <inertial>
-      <origin rpy="0 0 0" xyz="-0.0011186 -4.317E-05 0.26842"/>
-      <mass value="9.7333"/>
-      <inertia ixx="0.1750" ixy="0.0014142857" ixz="0.000885" iyy="0.183614285" iyz="0" izz="0.1541"/>
-    </inertial>
-    <visual>
-      <origin rpy="0 0 0" xyz="0 0 0"/>
-      <geometry>
-        <mesh filename="package://handsfree_gazebo/urdf_stone_v3/meshes/base_link.STL"/>
-      </geometry>
-      <material name="light_black"/>
-    </visual>
-    <collision>
-      <origin rpy="0 0 0" xyz="0 0 0"/>
-      <geometry>
-        <mesh filename="package://handsfree_gazebo/urdf_stone_v3/meshes/base_link.STL"/>
-      </geometry>
-    </collision>
-  </link>
-  <joint name="base_joint" type="fixed">
-    <origin xyz="0 0 0" rpy="0 0 0" />
-    <parent link="base_link"/>
-    <child link="base_footprint" />
-  </joint>
-  <link name="imu_link"/>
-  <joint name="imu_joint" type="fixed">
-    <origin xyz="0 0 0" rpy="0 0 0" />
-    <parent link="base_link"/>
-    <child link="imu_link" />
-  </joint>
-  <!--wheel left -->
-  <link name="wheel1_link">
-    <inertial>
-      <origin rpy="0 0 0" xyz="3.1631E-06 -7.2374E-08 -0.00032962"/>
-      <mass value="0.15338"/>
-      <inertia ixx="4.7342E-05" ixy="0" ixz="0" iyy="4.734E-05" iyz="0" izz="8.8619E-05"/>
-    </inertial>
-    <visual>
-      <origin rpy="0 0 0" xyz="0 0 0"/>
-      <geometry>
-        <mesh filename="package://handsfree_gazebo/urdf_stone_v3/meshes/wheel_left_link.STL"/>
-      </geometry>
-      <material name="">
-        <color rgba="1 0.94902 0.89804 1"/>
-      </material>
-    </visual>
-    <collision>
-      <origin rpy="0 0 0" xyz="0 0 0"/>
-      <geometry>
-        <mesh filename="package://handsfree_gazebo/urdf_stone_v3/meshes/wheel_left_link.STL"/>
-      </geometry>
-    </collision>
-  </link>
-  <joint name="wheel1_joint" type="continuous">
-    <origin rpy="-1.5708 0 0" xyz="0 0.1557 0.0124"/>
-    <parent link="base_link"/>
-    <child link="wheel1_link"/>
-    <axis xyz="0 0 1"/>
-    <limit effort="8.85" velocity="17.4" />
-  </joint>
-  <!--wheel right -->
-  <link name="wheel2_link">
-    <inertial>
-      <origin rpy="0 0 0" xyz="-3.1631E-06 -7.2862E-08 -0.00032962"/>
-      <mass value="0.15338"/>
-      <inertia ixx="4.7342E-05" ixy="0" ixz="0" iyy="4.734E-05" iyz="0" izz="8.8619E-05"/>
-    </inertial>
-    <visual>
-      <origin rpy="0 0 0" xyz="0 0 0"/>
-      <geometry>
-        <mesh filename="package://handsfree_gazebo/urdf_stone_v3/meshes/wheel_right_link.STL"/>
-      </geometry>
-      <material name="">
-        <color rgba="1 0.94902 0.89804 1"/>
-      </material>
-    </visual>
-    <collision>
-      <origin rpy="0 0 0" xyz="0 0 0"/>
-      <geometry>
-        <mesh filename="package://handsfree_gazebo/urdf_stone_v3/meshes/wheel_right_link.STL"/>
-      </geometry>
-    </collision>
-  </link>
-  <joint name="wheel2_joint" type="continuous">
-    <origin rpy="1.5708 0 0" xyz="0 -0.1557 0.0124"/>
-    <parent link="base_link"/>
-    <child link="wheel2_link"/>
-    <axis xyz="0 0 -1"/>
-    <limit effort="8.85" velocity="17.4" />
-  </joint>
-  <link name="caster_front_link">
-    <inertial>
-      <origin rpy="0 0 0" xyz="0.0048088 0.0096311 8.3348E-16"/>
-      <mass value="0.15338"/>
-      <inertia ixx="4.7342E-05" ixy="0" ixz="0" iyy="4.734E-05" iyz="0" izz="8.8619E-05"/>
-    </inertial>
-    <visual>
-      <origin rpy="0 0 0" xyz="0 0 0"/>
-      <geometry>
-        <sphere radius="0.032"/>
-      </geometry>
-      <material name="grey"/>
-    </visual>
-    <collision>
-      <geometry>
-        <sphere radius="0.032"/>
-      </geometry>
-      <origin rpy="0 0 0" xyz="0 0 0"/>
-    </collision>
-  </link>
-  <joint name="caster_front_joint" type="fixed">
-    <origin rpy="1.5708 0 0" xyz="0.126 0 0.0124"/>
-    <parent link="base_link"/>
-    <child link="caster_front_link"/>
-    <axis xyz="0 0 1"/>
-  </joint>
-  <link name="caster_back_link">
-    <inertial>
-      <origin rpy="0 0 0" xyz="-0.0048088 0.0096311 8.3433E-16"/>
-      <mass value="0.15338"/>
-      <inertia ixx="4.7342E-05" ixy="0" ixz="0" iyy="4.734E-05" iyz="0" izz="8.8619E-05"/>
-    </inertial>
-    <visual>
-      <origin rpy="0 0 0" xyz="0 0 0"/>
-      <geometry>
-        <sphere radius="0.032"/>
-      </geometry>
-      <material name="grey"/>
-    </visual>
-    <collision>
-      <geometry>
-        <sphere radius="0.032"/>
-      </geometry>
-      <origin rpy="0 0 0" xyz="0 0 0"/>
-    </collision>
-  </link>
-  <joint name="caster_back_joint" type="fixed">
-    <origin rpy="1.5708 0 0" xyz="-0.126 0 0.0124"/>
-    <parent link="base_link"/>
-    <child link="caster_back_link"/>
-    <axis xyz="0 0 1"/>
-  </joint>
-  <link name="laser_link">
-    <inertial>
-      <origin rpy="0 0 0" xyz="-0.00012709 4.6538E-05 -0.011453"/>
-      <mass value="0.13632"/>
-      <inertia ixx="7.1499E-05" ixy="0" ixz="0" iyy="7.1883E-05" iyz="0" izz="4.6678E-05"/>
-    </inertial>
-    <visual>
-      <origin rpy="0 0 0" xyz="0 0 0"/>
-      <geometry>
-        <mesh filename="package://handsfree_gazebo/urdf_stone_v3/meshes/laser_link.STL"/>
-      </geometry>
-      <material name="orange"/>
-    </visual>
-    <collision>
-      <origin rpy="0 0 0" xyz="0 0 0"/>
-      <geometry>
-        <mesh filename="package://handsfree_gazebo/urdf_stone_v3/meshes/laser_link.STL"/>
-      </geometry>
-    </collision>
-  </link>
-  <joint name="laser_joint" type="fixed">
-    <origin rpy="0 0 0" xyz="0.145 0 0.14203"/>
-    <parent link="base_link"/>
-    <child link="laser_link"/>
-    <axis xyz="0 0 0"/>
-  </joint>
-  <link name="yaw_link">
-    <inertial>
-      <origin rpy="0 0 0" xyz="8.5422E-05 0.0001613 0.0023545"/>
-      <mass value="0.15082"/>
-      <inertia ixx="0.00012558" ixy="0" ixz="0" iyy="0.00012402" iyz="0" izz="0.00023372"/>
-    </inertial>
-    <visual>
-      <origin rpy="0 0 0" xyz="0 0 0"/>
-      <geometry>
-        <mesh filename="package://handsfree_gazebo/urdf_stone_v3/meshes/yaw_link.STL"/>
-      </geometry>
-      <material name="">
-        <color rgba="0.89804 0.91765 0.92941 1"/>
-      </material>
-    </visual>
-    <collision>
-      <origin rpy="0 0 0" xyz="0 0 0"/>
-      <geometry>
-        <mesh filename="package://handsfree_gazebo/urdf_stone_v3/meshes/yaw_link.STL"/>
-      </geometry>
-    </collision>
-  </link>
-  <joint name="yaw_joint" type="revolute">
-    <origin rpy="0 0 0" xyz="0 0 0.894"/>
-    <parent link="base_link"/>
-    <child link="yaw_link"/>
-    <axis xyz="0 0 1"/>
-    <limit
-      upper="1"
-      lower="-1"
-      effort="0.03"
-      velocity="1" />
-  </joint>
-  <link name="pitch_link">
-    <inertial>
-      <origin rpy="0 0 0" xyz="-0.00024079 -0.041896 -9.1768E-05"/>
-      <mass value="0.06208"/>
-      <inertia ixx="4.7571E-05" ixy="0" ixz="0" iyy="2.3344E-05" iyz="0" izz="3.516E-05"/>
-    </inertial>
-    <visual>
-      <origin rpy="0 0 0" xyz="0 0 0"/>
-      <geometry>
-        <mesh filename="package://handsfree_gazebo/urdf_stone_v3/meshes/pitch_link.STL"/>
-      </geometry>
-      <material name="">
-        <color rgba="0.89804 0.91765 0.92941 1"/>
-      </material>
-    </visual>
-    <collision>
-      <origin rpy="0 0 0" xyz="0 0 0"/>
-      <geometry>
-        <mesh filename="package://handsfree_gazebo/urdf_stone_v3/meshes/pitch_link.STL"/>
-      </geometry>
-    </collision>
-  </link>
-  <joint name="pitch_joint" type="revolute">
-    <origin rpy="-1.5708 0 3.14159" xyz="0.01 5E-05 0.01475"/>
-    <parent link="yaw_link"/>
-    <child link="pitch_link"/>
-    <axis xyz="0 0 1"/>
-    <limit
-      upper="0.87"
-      lower="-0.52"
-      effort="0.03"
-      velocity="1" />
-  </joint>
-  <link name="camera_link">
-    <inertial>
-      <origin rpy="0 0 0" xyz="-0.017766 1.5798E-06 -0.00017508"/>
-      <mass value="0.15757"/>
-      <inertia ixx="0.00039792" ixy="0" ixz="0" iyy="2.4687E-05" iyz="0" izz="0.00040604"/>
-    </inertial>
-    <visual>
-      <origin rpy="0 0 0" xyz="0 0 0"/>
-      <geometry>
-        <mesh filename="package://handsfree_gazebo/urdf_stone_v3/meshes/xtion_link.STL"/>
-      </geometry>
-      <material name="">
-        <color rgba="0.33333 0.33333 0.33333 1"/>
-      </material>
-    </visual>
-    <collision>
-      <origin rpy="0 0 0" xyz="0 0 0"/>
-      <geometry>
-        <mesh filename="package://handsfree_gazebo/urdf_stone_v3/meshes/xtion_link.STL"/>
-      </geometry>
-    </collision>
-  </link>
-  <joint name="camera_joint" type="fixed">
-    <origin rpy="1.5708 3.14159 0" xyz="-0.0181 -0.08706 0.00011573"/>
-    <parent link="pitch_link"/>
-    <child link="camera_link"/>
-    <axis xyz="0 0 0"/>
-  </joint>
-  <!--for xtion sensor model -->
-      <joint name="camera_depth_joint" type="fixed">
-        <origin xyz="0.0 0.049 0.0" rpy="0 0 0" />
-        <parent link="camera_link" />
-        <child link="camera_depth_frame"/>
-      </joint>
-      <link name="camera_depth_frame"/>
-      <joint name="camera_depth_optical_joint" type="fixed">
-        <origin xyz="0 0 0" rpy="${-M_PI/2} 0.0 ${-M_PI/2}" />
-        <parent link="camera_depth_frame" />
-        <child link="camera_depth_optical_frame"/>
-      </joint>
-      <link name="camera_depth_optical_frame"/>
-      <joint name="camera_rgb_joint" type="fixed">
-        <origin xyz="0.0 0.022 0.0" rpy="0 0 0" />
-        <parent link="camera_link" />
-        <child link="camera_rgb_frame"/>
-      </joint>
-      <link name="camera_rgb_frame"/>
-      <joint name="camera_rgb_optical_joint" type="fixed">
-        <origin xyz="0 0 0" rpy="${-M_PI/2} 0.0 ${-M_PI/2}" />
-        <parent link="camera_rgb_frame" />
-        <child link="camera_rgb_optical_frame"/>
-      </joint>
-      <link name="camera_rgb_optical_frame"/>
+    <link name="base_footprint"/>
+    <link name="base_link">
+      <inertial>
+        <origin rpy="0 0 0" xyz="-0.0011186 -4.317E-05 0.26842"/>
+        <mass value="9.7333"/>
+        <inertia ixx="0.1750" ixy="0.0014142857" ixz="0.000885" iyy="0.183614285" iyz="0" izz="0.1541"/>
+      </inertial>
+      <visual>
+        <origin rpy="0 0 0" xyz="0.045 0 0.139"/>
+        <geometry>
+          <cylinder length="0.152" radius="0.115"/>
+        </geometry>
+        <material name="transparent_black">
+          <color rgba="0.4 0.4 0.4 0.7"/>
+        </material>
+      </visual>
+      <collision>
+        <origin rpy="0 0 0" xyz="0 0 0"/>
+        <geometry>
+          <mesh filename="package://handsfree_gazebo/urdf_stone_v3/meshes/base_link.STL"/>
+        </geometry>
+      </collision>
+    </link>
+    <joint name="base_joint" type="fixed">
+      <origin xyz="0 0 0" rpy="0 0 0" />
+      <parent link="base_link"/>
+      <child link="base_footprint" />
+    </joint>
+    <link name="imu_link"/>
+    <joint name="imu_joint" type="fixed">
+      <origin xyz="0.021 0.021 0.121" rpy="0 0.01 0" />
+      <parent link="base_link"/>
+      <child link="imu_link" />
+    </joint>
+    <!--wheel left -->
+    <link name="wheel1_link">
+      <inertial>
+        <origin rpy="0 0 0" xyz="3.1631E-06 -7.2374E-08 -0.00032962"/>
+        <mass value="0.15338"/>
+        <inertia ixx="4.7342E-05" ixy="0" ixz="0" iyy="4.734E-05" iyz="0" izz="8.8619E-05"/>
+      </inertial>
+      <visual>
+        <origin rpy="0 0 0" xyz="0 0 0"/>
+        <geometry>
+          <mesh filename="package://handsfree_gazebo/urdf_stone_v3/meshes/wheel_left_link.STL"/>
+        </geometry>
+        <material name="blue"/>
+      </visual>
+      <collision>
+        <origin rpy="0 0 0" xyz="0 0 0"/>
+        <geometry>
+          <mesh filename="package://handsfree_gazebo/urdf_stone_v3/meshes/wheel_left_link.STL"/>
+        </geometry>
+      </collision>
+    </link>
+    <joint name="wheel1_joint" type="continuous">
+      <origin rpy="-1.5708 0 0" xyz="0 0.1025 0.0325"/>
+      <parent link="base_link"/>
+      <child link="wheel1_link"/>
+      <axis xyz="0 0 1"/>
+      <limit effort="8.85" velocity="17.4" />
+    </joint>
+    <!--wheel right -->
+    <link name="wheel2_link">
+      <inertial>
+        <origin rpy="0 0 0" xyz="-3.1631E-06 -7.2862E-08 -0.00032962"/>
+        <mass value="0.15338"/>
+        <inertia ixx="4.7342E-05" ixy="0" ixz="0" iyy="4.734E-05" iyz="0" izz="8.8619E-05"/>
+      </inertial>
+      <visual>
+        <origin rpy="0 0 0" xyz="0 0 0"/>
+        <geometry>
+          <mesh filename="package://handsfree_gazebo/urdf_stone_v3/meshes/wheel_right_link.STL"/>
+        </geometry>
+        <material name="blue"/>
+      </visual>
+      <collision>
+        <origin rpy="0 0 0" xyz="0 0 0"/>
+        <geometry>
+          <mesh filename="package://handsfree_gazebo/urdf_stone_v3/meshes/wheel_right_link.STL"/>
+        </geometry>
+      </collision>
+    </link>
+    <joint name="wheel2_joint" type="continuous">
+      <origin rpy="1.5708 0 0" xyz="0 -0.1025 0.0325"/>
+      <parent link="base_link"/>
+      <child link="wheel2_link"/>
+      <axis xyz="0 0 -1"/>
+      <limit effort="8.85" velocity="17.4" />
+    </joint>
+    <link name="caster_front_link">
+      <inertial>
+        <origin rpy="0 0 0" xyz="0.0048088 0.0096311 8.3348E-16"/>
+        <mass value="0.15338"/>
+        <inertia ixx="4.7342E-05" ixy="0" ixz="0" iyy="4.734E-05" iyz="0" izz="8.8619E-05"/>
+      </inertial>
+      <visual>
+        <origin rpy="0 0 0" xyz="-0.025 0.0 0.0"/>
+        <geometry>
+          <mesh filename="package://handsfree_gazebo/urdf_stone_v3/meshes/caster_front_link.STL"/>
+        </geometry>
+        <material name="ivory">
+          <color rgba="0.8 0.8 0.75 1"/>
+        </material>
+      </visual>
+      <collision>
+        <geometry>
+          <sphere radius="0.032"/>
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