Commit message: add mini urdf

File: handsfree_gazebo/urdf/stone_v3/stone_v3_base.xacro (robot description, xacro)
@@ -5,5 +5,5 @@
 <!-- =================================================================================== -->
 <robot name="stone_v3_base"  xmlns:xacro="http://www.ros.org/wiki/xacro">
-  <xacro:include filename="$(find handsfree_gazebo)/urdf_stone_v3/common_properties.xacro"/>
+  <xacro:include filename="$(find handsfree_gazebo)/urdf/stone_v3/common_properties.xacro"/>
   <xacro:macro name="stone_v3_base">
   <link name="base_footprint"/>
@@ -17,5 +17,5 @@
       <origin rpy="0 0 0" xyz="0 0 0"/>
       <geometry>
-        <mesh filename="package://handsfree_gazebo/urdf_stone_v3/meshes/base_link.STL"/>
+        <mesh filename="package://handsfree_gazebo/urdf/stone_v3/meshes/base_link.STL"/>
       </geometry>
       <material name="light_black"/>
@@ -24,5 +24,5 @@
       <origin rpy="0 0 0" xyz="0 0 0"/>
       <geometry>
-        <mesh filename="package://handsfree_gazebo/urdf_stone_v3/meshes/base_link.STL"/>
+        <mesh filename="package://handsfree_gazebo/urdf/stone_v3/meshes/base_link.STL"/>
       </geometry>
     </collision>
@@ -49,5 +49,5 @@
       <origin rpy="0 0 0" xyz="0 0 0"/>
       <geometry>
-        <mesh filename="package://handsfree_gazebo/urdf_stone_v3/meshes/wheel_left_link.STL"/>
+        <mesh filename="package://handsfree_gazebo/urdf/stone_v3/meshes/wheel_left_link.STL"/>
       </geometry>
       <material name="">
@@ -58,5 +58,5 @@
       <origin rpy="0 0 0" xyz="0 0 0"/>
       <geometry>
-        <mesh filename="package://handsfree_gazebo/urdf_stone_v3/meshes/wheel_left_link.STL"/>
+        <mesh filename="package://handsfree_gazebo/urdf/stone_v3/meshes/wheel_left_link.STL"/>
       </geometry>
     </collision>
@@ -79,5 +79,5 @@
       <origin rpy="0 0 0" xyz="0 0 0"/>
       <geometry>
-        <mesh filename="package://handsfree_gazebo/urdf_stone_v3/meshes/wheel_right_link.STL"/>
+        <mesh filename="package://handsfree_gazebo/urdf/stone_v3/meshes/wheel_right_link.STL"/>
       </geometry>
       <material name="">
@@ -88,5 +88,5 @@
       <origin rpy="0 0 0" xyz="0 0 0"/>
       <geometry>
-        <mesh filename="package://handsfree_gazebo/urdf_stone_v3/meshes/wheel_right_link.STL"/>
+        <mesh filename="package://handsfree_gazebo/urdf/stone_v3/meshes/wheel_right_link.STL"/>
       </geometry>
     </collision>
@@ -160,5 +160,5 @@
       <origin rpy="0 0 0" xyz="0 0 0"/>
       <geometry>
-        <mesh filename="package://handsfree_gazebo/urdf_stone_v3/meshes/laser_link.STL"/>
+        <mesh filename="package://handsfree_gazebo/urdf/stone_v3/meshes/laser_link.STL"/>
       </geometry>
       <material name="orange"/>
@@ -167,5 +167,5 @@
       <origin rpy="0 0 0" xyz="0 0 0"/>
       <geometry>
-        <mesh filename="package://handsfree_gazebo/urdf_stone_v3/meshes/laser_link.STL"/>
+        <mesh filename="package://handsfree_gazebo/urdf/stone_v3/meshes/laser_link.STL"/>
       </geometry>
     </collision>
@@ -186,5 +186,5 @@
       <origin rpy="0 0 0" xyz="0 0 0"/>
       <geometry>
-        <mesh filename="package://handsfree_gazebo/urdf_stone_v3/meshes/yaw_link.STL"/>
+        <mesh filename="package://handsfree_gazebo/urdf/stone_v3/meshes/yaw_link.STL"/>
       </geometry>
       <material name="">
@@ -195,5 +195,5 @@
       <origin rpy="0 0 0" xyz="0 0 0"/>
       <geometry>
-        <mesh filename="package://handsfree_gazebo/urdf_stone_v3/meshes/yaw_link.STL"/>
+        <mesh filename="package://handsfree_gazebo/urdf/stone_v3/meshes/yaw_link.STL"/>
       </geometry>
     </collision>
@@ -219,5 +219,5 @@
       <origin rpy="0 0 0" xyz="0 0 0"/>
       <geometry>
-        <mesh filename="package://handsfree_gazebo/urdf_stone_v3/meshes/pitch_link.STL"/>
+        <mesh filename="package://handsfree_gazebo/urdf/stone_v3/meshes/pitch_link.STL"/>
       </geometry>
       <material name="">
@@ -228,5 +228,5 @@
       <origin rpy="0 0 0" xyz="0 0 0"/>
       <geometry>
-        <mesh filename="package://handsfree_gazebo/urdf_stone_v3/meshes/pitch_link.STL"/>
+        <mesh filename="package://handsfree_gazebo/urdf/stone_v3/meshes/pitch_link.STL"/>
       </geometry>
     </collision>
@@ -252,5 +252,5 @@
       <origin rpy="0 0 0" xyz="0 0 0"/>
       <geometry>
-        <mesh filename="package://handsfree_gazebo/urdf_stone_v3/meshes/xtion_link.STL"/>
+        <mesh filename="package://handsfree_gazebo/urdf/stone_v3/meshes/xtion_link.STL"/>
       </geometry>
       <material name="">
@@ -261,5 +261,5 @@
       <origin rpy="0 0 0" xyz="0 0 0"/>
       <geometry>
-        <mesh filename="package://handsfree_gazebo/urdf_stone_v3/meshes/xtion_link.STL"/>
+        <mesh filename="package://handsfree_gazebo/urdf/stone_v3/meshes/xtion_link.STL"/>
       </geometry>
     </collision>

File: handsfree_gazebo/urdf/stone_v3/urdf/stone_v3_base.urdf (robot description, URDF)
Before this commit: robot stone_v3_base, 9 links, 8 joints
Links:
- removed link wheel_left_link
- removed link wheel_right_link
- removed link xtion_link
- added link camera_link, mass 0.15757; collision mesh filename=package://handsfree_gazebo/urdf/stone_v3/meshes/xtion_link.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; visual mesh filename=package://handsfree_gazebo/urdf/stone_v3/meshes/xtion_link.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
- added link wheel1_link, mass 0.15338; collision mesh filename=package://handsfree_gazebo/urdf/stone_v3/meshes/wheel_left_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; visual mesh filename=package://handsfree_gazebo/urdf/stone_v3/meshes/wheel_left_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
- added link wheel2_link, mass 0.15338; collision mesh filename=package://handsfree_gazebo/urdf/stone_v3/meshes/wheel_right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; visual mesh filename=package://handsfree_gazebo/urdf/stone_v3/meshes/wheel_right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
- link base_link: geometry collision mesh filename=package://handsfree_gazebo/urdf/stone_v3/meshes/base_link.S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; visual mesh filename=package://handsfree_gazebo/urdf/stone_v3/meshes/base_link.S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
- link caster_back_link: geometry collision mesh filename=package://handsfree_gazebo/urdf/stone_v3/meshes/caster_back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; visual mesh filename=package://handsfree_gazebo/urdf/stone_v3/meshes/caster_back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
- link caster_front_link: geometry collision mesh filename=package://handsfree_gazebo/urdf/stone_v3/meshes/caster_fron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; visual mesh filename=package://handsfree_gazebo/urdf/stone_v3/meshes/caster_fron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
- link laser_link: geometry collision mesh filename=package://handsfree_gazebo/urdf/stone_v3/meshes/laser_link.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; visual mesh filename=package://handsfree_gazebo/urdf/stone_v3/meshes/laser_link.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
- link pitch_link: geometry collision mesh filename=package://handsfree_gazebo/urdf/stone_v3/meshes/pitch_link.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; visual mesh filename=package://handsfree_gazebo/urdf/stone_v3/meshes/pitch_link.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
- link yaw_link: geometry collision mesh filename=package://handsfree_gazebo/urdf/stone_v3/meshes/yaw_link.STL; visual mesh filename=package://handsfree_gazebo/urdf/stone_v3/meshes/yaw_link.STL
Joints:
- removed joint wheel_left_joint
- removed joint wheel_right_joint
- removed joint xtion_joint
- added joint camera_joint: type fixed, parent pitch_link, child camera_link, origin xyz=0.0181 -0.08706 0.00011573 rpy=1.5708 0 0, axis 0 0 0
- added joint wheel1_joint: type continuous, parent base_link, child wheel1_link, origin xyz=0 0.1557 0.0124 rpy=-1.5708 0 0, axis 0 0 1
- added joint wheel2_joint: type continuous, parent base_link, child wheel2_link, origin xyz=0 -0.1557 0.0124 rpy=1.5708 0 0, axis 0 0 -1
